File: drone_pdb.sch (KiCad schematic (older format))
At the start: 2 parts

Commit message: basic schematic
Parts:
- added J?: Batt_OUT, symbol Connector:Conn_01x02_Female
- added J?: PM_IN, symbol Connector:Conn_01x02_Male
- added J?: PM_OUT, symbol Connector:Conn_01x02_Female
- added J? (x6): Conn_01x03_Female, symbol Connector:Conn_01x03_Female
- added J? (x6): Conn_01x03_Male, symbol Connector:Conn_01x03_Male
- added U? (x5): JMT_BS30D_30A, symbol esc:JMT_BS30D_30A
- J?: value Conn_01x02_Male -> Batt_IN
Connections:
- net at U?.1 (Bat+): now also J?.1 (Pin_1), U?.1 (Bat+), U?.1 (Bat+), U?.1 (Bat+), U?.1 (Bat+), U?.1 (Bat+)
- net at U?.3 (GND): now also U?.4 (Bat-), J?.2 (Pin_2), U?.3 (GND), U?.3 (GND), U?.3 (GND), U?.3 (GND), U?.3 (GND), U?.4 (Bat-), U?.4 (Bat-), U?.4 (Bat-), U?.4 (Bat-), U?.4 (Bat-)
- net at U?.5 (A): now also J?.1 (Pin_1)
- net at U?.6 (B): now also J?.2 (Pin_2)
- net at U?.7 (C): now also J?.3 (Pin_3)
- net at J?.1 (Pin_1): now also J?.1 (Pin_1), J?.1 (Pin_1)
- net at J?.2 (Pin_2): now also J?.2 (Pin_2), J?.2 (Pin_2)
- new net: J?.1 (Pin_1), U?.5 (A) (x5)
- new net: J?.2 (Pin_2), U?.6 (B) (x5)
- new net: J?.3 (Pin_3), U?.7 (C) (x5)
Other:
- moved on the sheet: J?, U?

Commit message: Basic esc footprint
Parts:
- J? (x2): symbol Connector:Conn_01x02_Male -> drone_pdb-rescue:Conn_01x02_Male-Connector
- J? (x2): symbol Connector:Conn_01x02_Female -> drone_pdb-rescue:Conn_01x02_Female-Connector
- J?: value Conn_01x03_Female -> M1; symbol Connector:Conn_01x03_Female -> drone_pdb-rescue:Conn_01x03_Female-Connector
- J?: value Conn_01x03_Female -> M2; symbol Connector:Conn_01x03_Female -> drone_pdb-rescue:Conn_01x03_Female-Connector
- J?: value Conn_01x03_Female -> M3; symbol Connector:Conn_01x03_Female -> drone_pdb-rescue:Conn_01x03_Female-Connector
- J?: value Conn_01x03_Female -> M4; symbol Connector:Conn_01x03_Female -> drone_pdb-rescue:Conn_01x03_Female-Connector
- J?: value Conn_01x03_Female -> M5; symbol Connector:Conn_01x03_Female -> drone_pdb-rescue:Conn_01x03_Female-Connector
- J?: value Conn_01x03_Female -> M6; symbol Connector:Conn_01x03_Female -> drone_pdb-rescue:Conn_01x03_Female-Connector
- J?: value Conn_01x03_Male -> M1; symbol Connector:Conn_01x03_Male -> drone_pdb-rescue:Conn_01x03_Male-Connector
- J?: value Conn_01x03_Male -> M2; symbol Connector:Conn_01x03_Male -> drone_pdb-rescue:Conn_01x03_Male-Connector
- J?: value Conn_01x03_Male -> M3; symbol Connector:Conn_01x03_Male -> drone_pdb-rescue:Conn_01x03_Male-Connector
- J?: value Conn_01x03_Male -> M4; symbol Connector:Conn_01x03_Male -> drone_pdb-rescue:Conn_01x03_Male-Connector
- J?: value Conn_01x03_Male -> M5; symbol Connector:Conn_01x03_Male -> drone_pdb-rescue:Conn_01x03_Male-Connector
- J?: value Conn_01x03_Male -> M6; symbol Connector:Conn_01x03_Male -> drone_pdb-rescue:Conn_01x03_Male-Connector
Connections:
- net at J?.1 (Pin_1), U?.1 (Bat+), U?.1 (Bat+)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: now also J?.2 (Pin_2), J?.2 (Pin_2), J?.2 (Pin_2), J?.2 (Pin_2), J?.2 (Pin_2), J?.2 (Pin_2)
- net at U?.2 (PWM): now also J?.1 (Pin_1) (x6)
- net at J?.2 (Pin_2), U?.3 (GND), U?.3 (GND)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: now also J?.3 (Pin_3), J?.3 (Pin_3), J?.3 (Pin_3), J?.3 (Pin_3), J?.3 (Pin_3), J?.3 (Pin_3)
Other:
- moved on the sheet: J?
Changed lines of the file:
@@
 $EndComp
 $Comp
-L Connector:Conn_01x02_Male J?
+L drone_pdb-rescue:Conn_01x02_Male-Connector J?
 U 1 1 61718702
 P 1000 1950
@@
 $EndComp
 $Comp
-L Connector:Conn_01x02_Male J?
+L drone_pdb-rescue:Conn_01x02_Male-Connector J?
 U 1 1 6171F40F
 P 3550 800
@@
 	1650 2050 1450 2050
 $Comp
-L Connector:Conn_01x02_Female J?
+L drone_pdb-rescue:Conn_01x02_Female-Connector J?
 U 1 1 6171EB6B
 P 1850 1950
@@
 $EndComp
 $Comp
-L Connector:Conn_01x02_Female J?
+L drone_pdb-rescue:Conn_01x02_Female-Connector J?
 U 1 1 61725B09
 P 1850 2200
@@
 	4550 1300 4350 1300
 Wire Wire Line
-	4350 1300 4350 2350
+	4350 1300 4350 1650
 Wire Wire Line
 	4350 4450 4550 4450
@@
 Connection ~ 4350 3400
 Wire Wire Line
-	4350 3400 4350 4450
+	4350 3400 4350 3750
 Wire Wire Line
 	4550 2350 4350 2350
 Connection ~ 4350 2350
 Wire Wire Line
-	4350 2350 4350 3400
+	4350 2350 4350 2700
 Wire Wire Line
 	4550 1900 4500 1900
@@
 Connection ~ 4250 4000
 Wire Wire Line
-	4250 4000 4250 5050
+	4250 4000 4250 4900
 Connection ~ 4250 2950
 Wire Wire Line
-	4250 2950 4250 4000
+	4250 2950 4250 3850
 Wire Wire Line
 	4250 2950 4500 2950
@@
 Connection ~ 4250 1900
 Wire Wire Line
-	4250 1900 4250 2950
-Wire Wire Line
-	4250 900  4250 1900
-$Comp
-L Connector:Conn_01x03_Female J?
+	4250 1900 4250 2800
+Wire Wire Line
+	4250 900  4250 1750
+$Comp
+L drone_pdb-rescue:Conn_01x03_Female-Connector J?
 U 1 1 617496C2
 P 5750 1600
 F 0 "J?" H 5778 1626 50  0000 L CNN
-F 1 "Conn_01x03_Female" H 5778 1535 50  0000 L CNN
+F 1 "M1" H 5778 1535 50  0000 L CNN
 F 2 "" H 5750 1600 50  0001 C CNN
 F 3 "~" H 5750 1600 50  0001 C CNN
@@
 	5450 1800 5350 1800
 $Comp
-L Connector:Conn_01x03_Female J?
+L drone_pdb-rescue:Conn_01x03_Female-Connector J?
 U 1 1 6174BF8B
 P 5750 2650
 F 0 "J?" H 5778 2676 50  0000 L CNN
-F 1 "Conn_01x03_Female" H 5778 2585 50  0000 L CNN
+F 1 "M2" H 5778 2585 50  0000 L CNN
 F 2 "" H 5750 2650 50  0001 C CNN
 F 3 "~" H 5750 2650 50  0001 C CNN
@@
 	5450 2850 5350 2850
 $Comp
-L Connector:Conn_01x03_Female J?
+L drone_pdb-rescue:Conn_01x03_Female-Connector J?
 U 1 1 6174D549
 P 5750 3700
 F 0 "J?" H 5778 3726 50  0000 L CNN
-F 1 "Conn_01x03_Female" H 5778 3635 50  0000 L CNN
+F 1 "M3" H 5778 3635 50  0000 L CNN
 F 2 "" H 5750 3700 50  0001 C CNN
 F 3 "~" H 5750 3700 50  0001 C CNN
@@
 	5450 3900 5350 3900
 $Comp
-L Connector:Conn_01x03_Female J?
+L drone_pdb-rescue:Conn_01x03_Female-Connector J?
 U 1 1 6174E8B9
 P 5750 4750
 F 0 "J?" H 5778 4776 50  0000 L CNN
-F 1 "Conn_01x03_Female" H 5778 4685 50  0000 L CNN
+F 1 "M4" H 5778 4685 50  0000 L CNN
 F 2 "" H 5750 4750 50  0001 C CNN
 F 3 "~" H 5750 4750 50  0001 C CNN
@@
 Connection ~ 4350 5500
 Wire Wire Line
-	4350 5500 4350 6550
-Wire Wire Line
-	4350 4450 4350 5500
+	4350 5500 4350 5850
+Wire Wire Line
+	4350 4450 4350 4800
 Wire Wire Line
 	4250 7150 4500 7150
 Connection ~ 4250 6100
 Wire Wire Line
-	4250 6100 4250 7150
-Wire Wire Line
-	4250 5050 4250 6100
+	4250 6100 4250 7000
+Wire Wire Line
+	4250 5050 4250 5950
 Wire Wire Line
 	4250 6100 4500 6100
@@
 	4500 7150 4550 7150
 $Comp
-L Connector:Conn_01x03_Female J?
+L drone_pdb-rescue:Conn_01x03_Female-Connector J?
 U 1 1 617589AE
 P 5750 5800
 F 0 "J?" H 5778 5826 50  0000 L CNN
-F 1 "Conn_01x03_Female" H 5778 5735 50  0000 L CNN
+F 1 "M5" H 5778 5735 50  0000 L CNN
 F 2 "" H 5750 5800 50  0001 C CNN
 F 3 "~" H 5750 5800 50  0001 C CNN
@@
 	5450 6000 5350 6000
 $Comp
-L Connector:Conn_01x03_Female J?
+L drone_pdb-rescue:Conn_01x03_Female-Connector J?
 U 1 1 617589BB
 P 5750 6850
 F 0 "J?" H 5778 6876 50  0000 L CNN
-F 1 "Conn_01x03_Female" H 5778 6785 50  0000 L CNN
+F 1 "M6" H 5778 6785 50  0000 L CNN
 F 2 "" H 5750 6850 50  0001 C CNN
 F 3 "~" H 5750 6850 50  0001 C CNN
@@
 Connection ~ 4350 4450
 $Comp
-L Connector:Conn_01x03_Male J?
+L drone_pdb-rescue:Conn_01x03_Male-Connector J?
 U 1 1 6176825A
-P 2800 1750
-F 0 "J?" H 2908 2031 50  0000 C CNN
-F 1 "Conn_01x03_Male" H 2908 1940 50  0000 C CNN
-F 2 "" H 2800 1750 50  0001 C CNN
-F 3 "~" H 2800 1750 50  0001 C CNN
-	1    2800 1750
-	1    0    0    -1
-$EndComp
-$Comp
-L Connector:Conn_01x03_Male J?
+P 3750 1650
+F 0 "J?" H 3858 1931 50  0000 C CNN
+F 1 "M1" H 3858 1840 50  0000 C CNN
+F 2 "" H 3750 1650 50  0001 C CNN
+F 3 "~" H 3750 1650 50  0001 C CNN
+	1    3750 1650
+	1    0    0    -1
+$EndComp
+$Comp
+L drone_pdb-rescue:Conn_01x03_Male-Connector J?
 U 1 1 6176DEE7
-P 2800 2200
-F 0 "J?" H 2908 2481 50  0000 C CNN
-F 1 "Conn_01x03_Male" H 2908 2390 50  0000 C CNN
-F 2 "" H 2800 2200 50  0001 C CNN
-F 3 "~" H 2800 2200 50  0001 C CNN
-	1    2800 2200
-	1    0    0    -1
-$EndComp
-$Comp
-L Connector:Conn_01x03_Male J?
+P 3750 2700
+F 0 "J?" H 3858 2981 50  0000 C CNN
+F 1 "M2" H 3858 2890 50  0000 C CNN
+F 2 "" H 3750 2700 50  0001 C CNN
+F 3 "~" H 3750 2700 50  0001 C CNN
+	1    3750 2700
+	1    0    0    -1
+$EndComp
+$Comp
+L drone_pdb-rescue:Conn_01x03_Male-Connector J?
 U 1 1 617706AC
-P 2800 2650
-F 0 "J?" H 2908 2931 50  0000 C CNN
-F 1 "Conn_01x03_Male" H 2908 2840 50  0000 C CNN
-F 2 "" H 2800 2650 50  0001 C CNN
-F 3 "~" H 2800 2650 50  0001 C CNN
-	1    2800 2650
-	1    0    0    -1
-$EndComp
-$Comp
-L Connector:Conn_01x03_Male J?
+P 3750 3750
+F 0 "J?" H 3858 4031 50  0000 C CNN
+F 1 "M3" H 3858 3940 50  0000 C CNN
+F 2 "" H 3750 3750 50  0001 C CNN
+F 3 "~" H 3750 3750 50  0001 C CNN
+	1    3750 3750
+	1    0    0    -1
+$EndComp
+$Comp
+L drone_pdb-rescue:Conn_01x03_Male-Connector J?
 U 1 1 61779F26
-P 2800 3100
-F 0 "J?" H 2908 3381 50  0000 C CNN
-F 1 "Conn_01x03_Male" H 2908 3290 50  0000 C CNN
-F 2 "" H 2800 3100 50  0001 C CNN
-F 3 "~" H 2800 3100 50  0001 C CNN
-	1    2800 3100
-	1    0    0    -1
-$EndComp
-$Comp
-L Connector:Conn_01x03_Male J?
+P 3750 4800
+F 0 "J?" H 3858 5081 50  0000 C CNN
+F 1 "M4" H 3858 4990 50  0000 C CNN
+F 2 "" H 3750 4800 50  0001 C CNN
+F 3 "~" H 3750 4800 50  0001 C CNN
+	1    3750 4800
+	1    0    0    -1
+$EndComp
+$Comp
+L drone_pdb-rescue:Conn_01x03_Male-Connector J?
 U 1 1 61779F2C
-P 2800 3550
-F 0 "J?" H 2908 3831 50  0000 C CNN
-F 1 "Conn_01x03_Male" H 2908 3740 50  0000 C CNN
-F 2 "" H 2800 3550 50  0001 C CNN
-F 3 "~" H 2800 3550 50  0001 C CNN
-	1    2800 3550
-	1    0    0    -1
-$EndComp
-$Comp
-L Connector:Conn_01x03_Male J?
+P 3750 5850
+F 0 "J?" H 3858 6131 50  0000 C CNN
+F 1 "M5" H 3858 6040 50  0000 C CNN
+F 2 "" H 3750 5850 50  0001 C CNN
+F 3 "~" H 3750 5850 50  0001 C CNN
+	1    3750 5850
+	1    0    0    -1
+$EndComp
+$Comp
+L drone_pdb-rescue:Conn_01x03_Male-Connector J?
 U 1 1 61779F32
-P 2800 4000
-F 0 "J?" H 2908 4281 50  0000 C CNN
-F 1 "Conn_01x03_Male" H 2908 4190 50  0000 C CNN
-F 2 "" H 2800 4000 50  0001 C CNN
-F 3 "~" H 2800 4000 50  0001 C CNN
-	1    2800 4000
-	1    0    0    -1
-$EndComp
+P 3750 6900
+F 0 "J?" H 3858 7181 50  0000 C CNN
+F 1 "M6" H 3858 7090 50  0000 C CNN
+F 2 "" H 3750 6900 50  0001 C CNN
+F 3 "~" H 3750 6900 50  0001 C CNN
+	1    3750 6900
+	1    0    0    -1
+$EndComp
+Wire Wire Line
+	3950 1550 4550 1550
+Wire Wire Line
+	3950 1750 4250 1750
+Connection ~ 4250 1750
+Wire Wire Line
+	4250 1750 4250 1900
+Wire Wire Line
+	3950 1650 4350 1650
+Connection ~ 4350 1650
+Wire Wire Line
+	4350 1650 4350 2350
+Wire Wire Line
+	3950 2600 4550 2600
+Wire Wire Line
+	4350 2700 3950 2700
+Connection ~ 4350 2700
+Wire Wire Line
+	4350 2700 4350 3400
+Wire Wire Line
+	3950 2800 4250 2800
+Connection ~ 4250 2800
+Wire Wire Line
+	4250 2800 4250 2950
+Wire Wire Line
+	3950 3650 4550 3650
+Wire Wire Line
+	4350 3750 3950 3750
+Connection ~ 4350 3750
+Wire Wire Line
+	4350 3750 4350 4450
+Wire Wire Line
+	3950 3850 4250 3850
+Connection ~ 4250 3850
+Wire Wire Line
+	4250 3850 4250 4000
+Wire Wire Line
+	3950 4700 4550 4700
+Wire Wire Line
+	4350 4800 3950 4800
+Connection ~ 4350 4800
+Wire Wire Line
+	4350 4800 4350 5500
+Wire Wire Line
+	3950 4900 4250 4900
+Connection ~ 4250 4900
+Wire Wire Line
+	4250 4900 4250 5050
+Wire Wire Line
+	4550 5750 3950 5750
+Wire Wire Line
+	3950 5850 4350 5850
+Connection ~ 4350 5850
+Wire Wire Line
+	4350 5850 4350 6550
+Wire Wire Line
+	4250 5950 3950 5950
+Connection ~ 4250 5950
+Wire Wire Line
+	4250 5950 4250 6100
+Wire Wire Line
+	3950 6800 4550 6800
+Wire Wire Line
+	3950 6900 4350 6900
+Wire Wire Line
+	4350 6900 4350 6550
+Connection ~ 4350 6550
+Wire Wire Line
+	3950 7000 4250 7000
+Connection ~ 4250 7000
+Wire Wire Line
+	4250 7000 4250 7150
 $EndSCHEMATC

Commit message: Started pcb design
Parts:
- removed U? (x5): JMT_BS30D_30A, symbol esc:JMT_BS30D_30A
- added U1, U2, U4, U5, U6: JMT_BS30D_30A, esc:BS30D, symbol esc:JMT_BS30D_30A
- J1, J2, J3, J4: renamed from J?; footprint (none) -> Connector_AMASS:AMASS_XT60-M_1x02_P7.20mm_Vertical
- J10, J5, J6, J7, J8, J9: renamed from J?; footprint (none) -> Connector_PinHeader_2.54mm:PinHeader_1x03_P2.54mm_Vertical
- J11, J12, J13, J14, J15, J16: renamed from J?; footprint (none) -> Connector_AMASS:AMASS_MR30PW-FB_1x03_P3.50mm_Horizontal
- U3: renamed from U?; footprint (none) -> esc:BS30D
Connections:
- net at J10.2 (Pin_2), J4.1 (Pin_1), J5.2 (Pin_2)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: now also U1.1 (Bat+), U2.1 (Bat+), U4.1 (Bat+), U5.1 (Bat+), U6.1 (Bat+)
- net at J5.1 (Pin_1): now also U1.2 (PWM)
- net at J10.3 (Pin_3), J4.2 (Pin_2), J5.3 (Pin_3)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: now also U1.3 (GND), U1.4 (Bat-), U2.3 (GND), U2.4 (Bat-), U4.3 (GND), U4.4 (Bat-), U5.3 (GND), U5.4 (Bat-), U6.3 (GND), U6.4 (Bat-)
- net at J11.1 (Pin_1): now also U1.5 (A)
- net at J11.2 (Pin_2): now also U1.6 (B)
- net at J11.3 (Pin_3): now also U1.7 (C)
- net at J6.1 (Pin_1): now also U2.2 (PWM)
- net at J12.1 (Pin_1): now also U2.5 (A)
- net at J12.2 (Pin_2): now also U2.6 (B)
- net at J12.3 (Pin_3): now also U2.7 (C)
- net at J8.1 (Pin_1): now also U4.2 (PWM)
- net at J14.1 (Pin_1): now also U4.5 (A)
- net at J14.2 (Pin_2): now also U4.6 (B)
- net at J14.3 (Pin_3): now also U4.7 (C)
- net at J9.1 (Pin_1): now also U5.2 (PWM)
- net at J15.1 (Pin_1): now also U5.5 (A)
- net at J15.2 (Pin_2): now also U5.6 (B)
- net at J15.3 (Pin_3): now also U5.7 (C)
- net at J10.1 (Pin_1): now also U6.2 (PWM)
- net at J16.1 (Pin_1): now also U6.5 (A)
- net at J16.2 (Pin_2): now also U6.6 (B)
- net at J16.3 (Pin_3): now also U6.7 (C)
